File: OPTIGA_Trust_M_Module.kicad_pcb (KiCad board)
At the start: 2 copper layers, 25.4 x 25.4 mm, 13 parts, among them J1 Conn_01x08, Q1 PMOS, Q2 NMOS, U1 SLS32AIA

Commit message: modify: uson-10 footprint
Other:
- board text added: "Naisu / 20240429"
- board text removed: "Naisu / 20240424"
Changed lines of the file:
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@@
 			)
 		)
-		(sheetname "根目录")
-		(sheetfile "OPTIGA_Trust_M_Module.kicad_sch")
 		(attr smd)
 		(fp_line
@@
 		)
 		(pad "1" smd roundrect
-			(at -1.3 -1)
+			(at -1.375 -1)
 			(size 0.6 0.25)
 			(layers "F.Cu" "F.Paste" "F.Mask")
@@
 		)
 		(pad "2" smd roundrect
-			(at -1.3 -0.5)
+			(at -1.375 -0.5)
 			(size 0.6 0.25)
 			(layers "F.Cu" "F.Paste" "F.Mask")
@@
 		)
 		(pad "3" smd roundrect
-			(at -1.3 0)
+			(at -1.375 0)
 			(size 0.6 0.25)
 			(layers "F.Cu" "F.Paste" "F.Mask")
@@
 		)
 		(pad "4" smd roundrect
-			(at -1.3 0.5)
+			(at -1.375 0.5)
 			(size 0.6 0.25)
 			(layers "F.Cu" "F.Paste" "F.Mask")
@@
 		)
 		(pad "5" smd roundrect
-			(at -1.3 1)
+			(at -1.375 1)
 			(size 0.6 0.25)
 			(layers "F.Cu" "F.Paste" "F.Mask")
@@
 		)
 		(pad "6" smd roundrect
-			(at 1.3 1)
+			(at 1.375 1)
 			(size 0.6 0.25)
 			(layers "F.Cu" "F.Paste" "F.Mask")
@@
 		)
 		(pad "7" smd roundrect
-			(at 1.3 0.5)
+			(at 1.375 0.5)
 			(size 0.6 0.25)
 			(layers "F.Cu" "F.Paste" "F.Mask")
@@
 		)
 		(pad "8" smd roundrect
-			(at 1.3 0)
+			(at 1.375 0)
 			(size 0.6 0.25)
 			(layers "F.Cu" "F.Paste" "F.Mask")
@@
 		)
 		(pad "9" smd roundrect
-			(at 1.3 -0.5)
+			(at 1.375 -0.5)
 			(size 0.6 0.25)
 			(layers "F.Cu" "F.Paste" "F.Mask")
@@
 		)
 		(pad "10" smd roundrect
-			(at 1.3 -1)
+			(at 1.375 -1)
 			(size 0.6 0.25)
 			(layers "F.Cu" "F.Paste" "F.Mask")
@@
 			)
 		)
-		(property "Footprint" ""
+		(property "Footprint" "0_ungrouped:logo-nx_4.0x3.0mm"
 			(at 0 0 0)
 			(unlocked yes)
@@
 		)
 	)
-	(gr_text "Naisu / 20240424"
+	(gr_text "Naisu / 20240429"
 		(at 135.763 102.616 0)
 		(layer "F.SilkS")
